File: Hardware/PCB/Electronic Leadscrew.kicad_sch (KiCad schematic)
At the start: 26 parts, among them J101 DISPLAY, J102 ENCODER, J103 STEPPER DRIVER, Q101 SI2302, Q102 SI2302, Q103 SI2302, U101 PI PICO, U102 TPT480L1-SO1R, U103 SDB628

Commit message: Update PCB
Parts:
- removed J102: ENCODER, Connector_Dsub:DSUB-9_Female_Horizontal_P2.77x2.84mm_EdgePinOffset4.94mm_Housed_MountingHolesOffset7.48mm, symbol Connector:DE9_Receptacle
- removed R101, R102, R105, R106: 0R, symbol Device:R
- added J102: ENCODER, Connector_Dsub:DSUB-9_Male_Horizontal_P2.77x2.84mm_EdgePinOffset7.70mm_Housed_MountingHolesOffset9.12mm, symbol Connector:DE9_Plug
- J101: footprint Connector_Dsub:DSUB-9_Female_Horizontal_P2.77x2.84mm_EdgePinOffset4.94mm_Housed_MountingHolesOffset7.48mm -> Connector_Dsub:DSUB-9_Female_Horizontal_P2.77x2.84mm_EdgePinOffset7.70mm_Housed_MountingHolesOffset9.12mm
- J103: footprint TerminalBlock:TerminalBlock_Xinya_XY308-2.54-4P_1x04_P2.54mm_Horizontal -> TerminalBlock_4Ucon:TerminalBlock_4Ucon_1x04_P3.50mm_Horizontal
Connections:
- net STP_DIR+ is gone; now on net +5V: J103.3 (Pin_3)
- net STP_PUL+ is gone; now on net +5V: J103.1 (Pin_1)
- net +12V: now also J102.1
- net ENC_CLK: now also U101.24 (GP18); no longer U101.21 (GP16)
- net ENC_CLK+: now also J102.2
- net ENC_CLK-: now also J102.3
- net ENC_DAT: now also U101.21 (GP16); no longer U101.24 (GP18)
- net ENC_DAT+: now also J102.5
- net ENC_DAT-: now also J102.4
- net GND: now also J102.6, J102.7, J102.8
- net ~{ENC_STAT}: now also J102.9
- removed net NC: J101.2, J101.4, J101.5, J101.9
Other:
- moved on the sheet: J103
